Commit message: Modified Parameters

File: assets/fingerik/finger.urdf (robot description, URDF)
Before this commit: robot None, 10 links, 9 joints
Links:
- link 0-dual_servo_shell: geometry collision mesh filename=./mesh/dual_servo_shell.obj scale=0.001 0.001 0.001; visual mesh filename=./mesh/dual_servo_shell.obj scale=0.001 0.001 0.001
