Commit message: Use closed environment to avoid cubes from escaping out of the workspace

File: assets/quadfinger/robot_properties_fingers/urdf/high_table_boundary.urdf (robot description, URDF)
Before this commit: robot stage, 1 links, 0 joints
Links:
- link stage_link: geometry collision mesh filename=package://robot_properties_fingers/meshes/side_boundary.stl scale=0.001 0.001 0.001; visual mesh filename=package://robot_properties_fingers/meshes/side_boundary_vis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 scale=0.001 0.001 0.001

Commit message: Using negative goal position reward

File: assets/quadfinger/robot_properties_fingers/urdf/high_table_boundary.urdf (robot description, URDF)
Before this commit: robot stage, 1 links, 0 joints
Links:
- link stage_link: geometry collision mesh filename=package://robot_properties_fingers/meshes/high_table_bounda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 scale=1 1 1; visual mesh filename=package://robot_properties_fingers/meshes/high_table_bounda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 scale=1 1 1
