Commit message: Modified parameters

File: assets/quadfinger/gripper.urdf (robot description, URDF)
Before this commit: robot None, 38 links, 37 joints
Joints:
- joint 0-dof2: limit lower=-3.14159265 upper=3.14159265 effort=1000 velocity=1000 -> lower=-1.570796325 upper=1.570796325 effort=1000 velocity=1000
- joint 0-dof3: limit lower=-3.14159265 upper=3.14159265 effort=1000 velocity=1000 -> lower=-2.3561944875 upper=2.3561944875 effort=1000 velocity=1000
- joint 0-module_to_parent: origin xyz=-0.12 0 0 rpy=3.14159265 0 1.570796325 -> xyz=-0.1 0 0 rpy=3.14159265 0 1.570796325
- joint 1-dof2: limit lower=-3.14159265 upper=3.14159265 effort=1000 velocity=1000 -> lower=-1.570796325 upper=1.570796325 effort=1000 velocity=1000
- joint 1-dof3: limit lower=-3.14159265 upper=3.14159265 effort=1000 velocity=1000 -> lower=-2.3561944875 upper=2.3561944875 effort=1000 velocity=1000
- joint 1-module_to_parent: origin xyz=0 -0.12 0 rpy=3.14159265 0 3.14159265 -> xyz=0 -0.1 0 rpy=3.14159265 0 3.14159265
- joint 2-dof2: limit lower=-3.14159265 upper=3.14159265 effort=1000 velocity=1000 -> lower=-1.570796325 upper=1.570796325 effort=1000 velocity=1000
- joint 2-dof3: limit lower=-3.14159265 upper=3.14159265 effort=1000 velocity=1000 -> lower=-2.3561944875 upper=2.3561944875 effort=1000 velocity=1000
- joint 2-module_to_parent: origin xyz=0.12 0 0 rpy=3.14159265 0 -1.570796325 -> xyz=0.1 0 0 rpy=3.14159265 0 -1.570796325
- joint 3-dof2: limit lower=-3.14159265 upper=3.14159265 effort=1000 velocity=1000 -> lower=-1.570796325 upper=1.570796325 effort=1000 velocity=1000
- joint 3-dof3: limit lower=-3.14159265 upper=3.14159265 effort=1000 velocity=1000 -> lower=-2.3561944875 upper=2.3561944875 effort=1000 velocity=1000
- joint 3-module_to_parent: origin xyz=0 0.12 0 rpy=3.14159265 0 0 -> xyz=0 0.1 0 rpy=3.14159265 0 0

File: assets/quadfinger/module.urdf.xacro (robot description, xacro)
@@ -53,5 +53,5 @@
             <child link="${module_prefix}-finger1"/>
             <axis xyz="0 0 -1"/>
-            <limit effort="1000" lower="${-1*PI}" upper="${PI}" velocity="1000"/>
+            <limit effort="1000" lower="${-1*PI/2}" upper="${PI/2}" velocity="1000"/>
             <origin xyz="0 0 0.0368" rpy="0 0 0"/>
         </joint>
@@ -60,5 +60,5 @@
             <child link="${module_prefix}-finger2"/>
             <axis xyz="0 0 -1"/>
-            <limit effort="1000" lower="${-1*PI}" upper="${PI}" velocity="1000"/>
+            <limit effort="1000" lower="${-3*PI/4}" upper="${3*PI/4}" velocity="1000"/>
             <origin xyz="-0.0014142 -0.1 0.0014142" rpy="0 ${-1*PI/4.0} 0"/>
         </joint>

File: assets/quadfinger/quad_finger.urdf.xacro (robot description, xacro)
@@ -3,5 +3,5 @@
     <!--Import parts from xacro file-->
     <xacro:include filename="module.urdf.xacro"/>
-    <xacro:property name="radius" value="0.12"/>
+    <xacro:property name="radius" value="0.1"/>
     <link name="dummy">
         <inertial>

Commit message: Update simplified mesh models

File: assets/quadfinger/gripper.urdf (robot description, URDF)
Before this commit: robot None, 38 links, 37 joints
Links:
- link 0-base_motor_frame: geometry collision mesh filename=./mesh/base_motor_frame_simplified.stl scale=0.001 0.001 0.001; visual mesh filename=./mesh/base_motor_frame_simplified.stl scale=0.001 0.001 0.001
- link 0-dual_servo_shell: geometry collision mesh filename=./mesh/dual_servo_shell_simplified.obj scale=0.001 0.001 0.001; visual mesh filename=./mesh/dual_servo_shell_simplified.obj scale=0.001 0.001 0.001
- link 0-xm430_0: geometry collision mesh filename=./mesh/XM430-simplified.obj scale=0.001 0.001 0.001; visual mesh filename=./mesh/XM430-simplified.obj scale=0.001 0.001 0.001
- link 0-xm430_1: geometry collision mesh filename=./mesh/XM430-simplified.obj scale=0.001 0.001 0.001; visual mesh filename=./mesh/XM430-simplified.obj scale=0.001 0.001 0.001
- link 0-xm430_2: geometry collision mesh filename=./mesh/XM430-simplified.obj scale=0.001 0.001 0.001; visual mesh filename=./mesh/XM430-simplified.obj scale=0.001 0.001 0.001
- link 1-base_motor_frame: geometry collision mesh filename=./mesh/base_motor_frame_simplified.stl scale=0.001 0.001 0.001; visual mesh filename=./mesh/base_motor_frame_simplified.stl scale=0.001 0.001 0.001
- link 1-dual_servo_shell: geometry collision mesh filename=./mesh/dual_servo_shell_simplified.obj scale=0.001 0.001 0.001; visual mesh filename=./mesh/dual_servo_shell_simplified.obj scale=0.001 0.001 0.001
- link 1-xm430_0: geometry collision mesh filename=./mesh/XM430-simplified.obj scale=0.001 0.001 0.001; visual mesh filename=./mesh/XM430-simplified.obj scale=0.001 0.001 0.001
- link 1-xm430_1: geometry collision mesh filename=./mesh/XM430-simplified.obj scale=0.001 0.001 0.001; visual mesh filename=./mesh/XM430-simplified.obj scale=0.001 0.001 0.001
- link 1-xm430_2: geometry collision mesh filename=./mesh/XM430-simplified.obj scale=0.001 0.001 0.001; visual mesh filename=./mesh/XM430-simplified.obj scale=0.001 0.001 0.001
- link 2-base_motor_frame: geometry collision mesh filename=./mesh/base_motor_frame_simplified.stl scale=0.001 0.001 0.001; visual mesh filename=./mesh/base_motor_frame_simplified.stl scale=0.001 0.001 0.001
- link 2-dual_servo_shell: geometry collision mesh filename=./mesh/dual_servo_shell_simplified.obj scale=0.001 0.001 0.001; visual mesh filename=./mesh/dual_servo_shell_simplified.obj scale=0.001 0.001 0.001
- link 2-xm430_0: geometry collision mesh filename=./mesh/XM430-simplified.obj scale=0.001 0.001 0.001; visual mesh filename=./mesh/XM430-simplified.obj scale=0.001 0.001 0.001
- link 2-xm430_1: geometry collision mesh filename=./mesh/XM430-simplified.obj scale=0.001 0.001 0.001; visual mesh filename=./mesh/XM430-simplified.obj scale=0.001 0.001 0.001
- link 2-xm430_2: geometry collision mesh filename=./mesh/XM430-simplified.obj scale=0.001 0.001 0.001; visual mesh filename=./mesh/XM430-simplified.obj scale=0.001 0.001 0.001
- link 3-base_motor_frame: geometry collision mesh filename=./mesh/base_motor_frame_simplified.stl scale=0.001 0.001 0.001; visual mesh filename=./mesh/base_motor_frame_simplified.stl scale=0.001 0.001 0.001
- link 3-dual_servo_shell: geometry collision mesh filename=./mesh/dual_servo_shell_simplified.obj scale=0.001 0.001 0.001; visual mesh filename=./mesh/dual_servo_shell_simplified.obj scale=0.001 0.001 0.001
- link 3-xm430_0: geometry collision mesh filename=./mesh/XM430-simplified.obj scale=0.001 0.001 0.001; visual mesh filename=./mesh/XM430-simplified.obj scale=0.001 0.001 0.001
- link 3-xm430_1: geometry collision mesh filename=./mesh/XM430-simplified.obj scale=0.001 0.001 0.001; visual mesh filename=./mesh/XM430-simplified.obj scale=0.001 0.001 0.001
- link 3-xm430_2: geometry collision mesh filename=./mesh/XM430-simplified.obj scale=0.001 0.001 0.001; visual mesh filename=./mesh/XM430-simplified.obj scale=0.001 0.001 0.001

File: assets/quadfinger/parts.urdf.xacro (robot description, xacro)
@@ -67,5 +67,5 @@
                 <origin xyz="0.0 0.0 0.0" rpy="0.0 0.0 0.0"/>
                 <geometry>
-                    <mesh filename="${root_folder}/mesh/xm430.obj" scale="${scale}"/>
+                    <mesh filename="${root_folder}/mesh/XM430-simplified.obj" scale="${scale}"/>
                 </geometry>
             </visual>
@@ -73,5 +73,5 @@
                 <origin xyz="0.0 0.0 0.0" rpy="0.0 0.0 0.0"/>
                 <geometry>
-                    <mesh filename="${root_folder}/mesh/xm430.obj" scale="${scale}"/>
+                    <mesh filename="${root_folder}/mesh/XM430-simplified.obj" scale="${scale}"/>
                 </geometry>
             </collision>
@@ -84,5 +84,5 @@
                 <origin xyz="0 0 0" rpy="0 0 0"/>
                 <geometry>
-                    <mesh filename="${root_folder}/mesh/base_motor_frame.obj" scale="${scale}"/>
+                    <mesh filename="${root_folder}/mesh/base_motor_frame_simplified.stl" scale="${scale}"/>
                 </geometry>
             </visual>
@@ -90,5 +90,5 @@
                 <origin xyz="0 0 0" rpy="0 0 0"/>
                 <geometry>
-                    <mesh filename="${root_folder}/mesh/base_motor_frame.obj" scale="${scale}"/>
+                    <mesh filename="${root_folder}/mesh/base_motor_frame_simplified.stl" scale="${scale}"/>
                 </geometry>
             </collision>
@@ -101,5 +101,5 @@
                 <origin xyz="0.0 0.0 0.0" rpy="0.0 0.0 0.0"/>
                 <geometry>
-                    <mesh filename="${root_folder}/mesh/dual_servo_shell.obj" scale="${scale}"/>
+                    <mesh filename="${root_folder}/mesh/dual_servo_shell_simplified.obj" scale="${scale}"/>
                 </geometry>
             </visual>
@@ -107,5 +107,5 @@
                 <origin xyz="0.0 0.0 0.0" rpy="0.0 0.0 0.0"/>
                 <geometry>
-                    <mesh filename="${root_folder}/mesh/dual_servo_shell.obj" scale="${scale}"/>
+                    <mesh filename="${root_folder}/mesh/dual_servo_shell_simplified.obj" scale="${scale}"/>
                 </geometry>
             </collision>

File: assets/quadfinger_plate/gripper.urdf (robot description, URDF)
Before this commit: robot None, 38 links, 37 joints
Joints:
- joint z_offset: origin xyz=0 0 0.3 rpy=0 0 0 -> xyz=0 0 0.5 rpy=0 0 0

File: assets/quadfinger_plate/quad_finger.urdf.xacro (robot description, xacro)
@@ -19,5 +19,5 @@
         <parent link="dummy"/>
         <child link="z_offset_link"/>
-        <origin xyz="0 0 0.3" rpy="0 0 0"/>
+        <origin xyz="0 0 0.5" rpy="0 0 0"/>
     </joint>
     <!-->
