Commit message: Reversed dof3 direction

File: assets/quadfinger_plate/gripper.urdf (robot description, URDF)
Before this commit: robot None, 38 links, 37 joints
Joints:
- joint 0-dof3: axis 0 0 -1 -> 0 0 1
- joint 1-dof3: axis 0 0 -1 -> 0 0 1
- joint 2-dof3: axis 0 0 -1 -> 0 0 1
- joint 3-dof3: axis 0 0 -1 -> 0 0 1

File: assets/quadfinger_plate/module.urdf.xacro (robot description, xacro)
@@ -59,5 +59,5 @@
             <parent link="${module_prefix}-finger1"/>
             <child link="${module_prefix}-finger2"/>
-            <axis xyz="0 0 -1"/>
+            <axis xyz="0 0 1"/>
             <limit effort="1000" lower="${-3*PI/4}" upper="${3*PI/4}" velocity="1000"/>
             <origin xyz="-0.0014142 -0.1 0.0014142" rpy="0 ${-1*PI/4.0} 0"/>
