Commit message: Change dualfinger task plate to a smaller one

File: assets/dualfinger_plate/plate_color.urdf (robot description, URDF)
Before this commit: robot None, 3 links, 2 joints
Links:
- link front: mass None -> 0.5; geometry collision box size=0.3 0.15 0.006; visual box size=0.3 0.15 0.006
- link rear: mass None -> 0.5; geometry collision box size=0.3 0.15 0.006; visual box size=0.3 0.15 0.006

File: assets/dualfinger_plate/plate_color.urdf.xacro (robot description, xacro)
@@ -1,8 +1,8 @@
 <?xml version="1.0"?>
 <robot xmlns:xacro="http://www.ros.org/wiki/xacro">
-    <xacro:property name="side_length" value="0.4"/>
-    <xacro:property name="thickness" value="0.01"/>
+    <xacro:property name="side_length" value="0.3"/>
+    <xacro:property name="thickness" value="0.006"/>
     <xacro:property name="a_color_value" value="1.0"/>
-    <xacro:property name="density" value="1000"/>
+    <xacro:property name="mass" value="0.5"/>
     <material name="front_material">
         <color rgba="0.5 0.2 0.2 ${a_color_value}"/>
@@ -27,5 +27,5 @@
         </collision>
         <inertial>
-            <density value="${density}"/>
+            <mass value="${mass}"/>
         </inertial>
     </link>
@@ -45,5 +45,5 @@
         </collision>
         <inertial>
-            <density value="${density}"/>
+            <mass value="${mass}"/>
         </inertial>
     </link>
