Commit message: Zero the unreasonable reward term

File: assets/dualfinger_plate/dual_finger.urdf.xacro (robot description, xacro)
@@ -19,5 +19,5 @@
         <parent link="dummy"/>
         <child link="z_offset_link"/>
-        <origin xyz="0 0 0.33" rpy="0 0 0"/>
+        <origin xyz="0 0 0.30" rpy="0 0 0"/>
     </joint>
     <!-->

File: assets/dualfinger_plate/gripper.urdf (robot description, URDF)
Before this commit: robot None, 20 links, 19 joints
Joints:
- joint z_offset: origin xyz=0 0 0.33 rpy=0 0 0 -> xyz=0 0 0.30 rpy=0 0 0

Commit message: Modified friction coefficient

File: assets/dualfinger_plate/dual_finger.urdf.xacro (robot description, xacro)
@@ -3,5 +3,5 @@
     <!--Import parts from xacro file-->
     <xacro:include filename="module.urdf.xacro"/>
-    <xacro:property name="radius" value="0.1"/>
+    <xacro:property name="radius" value="0.2"/>
     <link name="dummy">
         <inertial>

File: assets/dualfinger_plate/plate_color.urdf (robot description, URDF)
Before this commit: robot None, 3 links, 2 joints
Links:
- link front: mass 0.5 -> 0.1
- link rear: mass 0.5 -> 0.1

File: assets/dualfinger_plate/plate_color.urdf.xacro (robot description, xacro)
@@ -4,5 +4,5 @@
     <xacro:property name="thickness" value="0.006"/>
     <xacro:property name="a_color_value" value="1.0"/>
-    <xacro:property name="mass" value="0.5"/>
+    <xacro:property name="mass" value="0.1"/>
     <material name="front_material">
         <color rgba="0.5 0.2 0.2 ${a_color_value}"/>
