Commit message: Add quadruped falling and knee touching ground reset and penalty

File: assets/module/module_xacro/overconstrained_left.urdf.xacro (robot description, xacro)
@@ -235,4 +235,14 @@
             <origin xyz="0.004243 -0.127 -0.005243" rpy="0 0 0"/>
         </joint>
+        <link name="${module_prefix}-knee_frame">
+            <geometry>
+                <origin xyz="0 0 0" rpy="0 0 0"/>
+            </geometry>
+        </link>
+        <joint name="${module_prefix}-knee_frame_fix" type="fixed">
+            <parent link="${module_prefix}-finger2"/>
+            <child link="${module_prefix}-knee_frame"/>
+            <origin xyz="0 0 0" rpy="0 0 0"/>
+        </joint>
     </xacro:macro>
 </robot>

File: assets/module/module_xacro/overconstrained_right.urdf.xacro (robot description, xacro)
@@ -235,4 +235,14 @@
             <origin xyz="-0.004243 -0.127 -0.005243" rpy="0 0 0"/>
         </joint>
+        <link name="${module_prefix}-knee_frame">
+            <geometry>
+                <origin xyz="0 0 0" rpy="0 0 0"/>
+            </geometry>
+        </link>
+        <joint name="${module_prefix}-knee_frame_fix" type="fixed">
+            <parent link="${module_prefix}-finger2"/>
+            <child link="${module_prefix}-knee_frame"/>
+            <origin xyz="0 0 0" rpy="0 0 0"/>
+        </joint>
     </xacro:macro>
 </robot>

File: assets/module/quadruped.urdf (robot description, URDF)
Before this commit: robot None, 39 links, 38 joints
Links:
- added link 0-knee_frame
- added link 1-knee_frame
- added link 2-knee_frame
- added link 3-knee_frame
Joints:
- added joint 0-knee_frame_fix: type fixed, parent 0-finger2, child 0-knee_frame, origin xyz=0 0 0 rpy=0 0 0
- added joint 1-knee_frame_fix: type fixed, parent 1-finger2, child 1-knee_frame, origin xyz=0 0 0 rpy=0 0 0
- added joint 2-knee_frame_fix: type fixed, parent 2-finger2, child 2-knee_frame, origin xyz=0 0 0 rpy=0 0 0
- added joint 3-knee_frame_fix: type fixed, parent 3-finger2, child 3-knee_frame, origin xyz=0 0 0 rpy=0 0 0
