Commit message: Parameter changes to improve trained policies

File: assets/module/quadruped.urdf (robot description, URDF)
Before this commit: robot None, 43 links, 42 joints
Links:
- link robot_base: mass 0.2 -> 0.4

File: assets/module/quadruped/overconstrained_horizontal_quadruped.urdf.xacro (robot description, xacro)
@@ -54,5 +54,5 @@
         </collision>
         <inertial>
-            <mass value="0.2"/>
+            <mass value="0.4"/>
         </inertial>
     </link>
